File: attiny-breakout-example/attiny-breakout.brd (EAGLE design)
At the start: 63 x 43 mm, 14 parts, among them J1 AVR_SPI_PROG_3X2NS, J2 CONN-11752, U1 3.3V/150mA

Commit message: Latest bits of the attiny breakout board, and the color sensors library.
Parts:
- added C6: 100n\, rcl:C0805
- added R2, R3: 4.7k, rcl:R0805
- added U2: VEML6040, color-sensors:VEML6040
- U$1: value ATTINY84ATTINY84-20MU -> ATTINY84-20MU
- U1: value 3.3V/150mA -> MIC5025-3.3V
Connections:
- net N$10 renamed PB0
- net N$11 renamed PA7
- net N$12 renamed PA3
- net N$13 renamed PA2
- net N$14 renamed PA1
- net N$15 renamed PA0
- net N$3 renamed MISO
- net N$4 renamed !RESET
- net N$8 renamed PB2
- net N$9 renamed PB1
- removed net N$1: J1.3, JP1.9, U$1.1
- removed net N$2: J1.4, JP1.7, U$1.16
- new net MOSI: J1.4, JP1.7, R3.1, U$1.16, U2.2
- new net SCL: J1.3, JP1.9, R2.1, U$1.1, U2.3
- net 3.3V: now also C6.1, R2.2, R3.2, U2.4
- net GND: now also C6.2, U2.1
Routing:
- net 3.3V: track 5.10 -> 30.2 mm
- net GND: track 36.6 -> 20.3 mm, vias 2 -> 12
- net PA1: track 0.00 -> 5.03 mm, vias 0 -> 2
- net PA2: track 0.00 -> 1.79 mm
- added copper zone on layer 1, net GND
- added copper zone on layer 16, net GND

Commit message: Not sure why this isn't committed, so here you go.
Parts:
- moved TP3 1.20 mm to (17.3, 10.2)
- moved C4 1.10 mm to (17.3, 7.00)
- moved TP2 0.66 mm to (7.60, 10.4)
- moved R1 0.51 mm to (9.90, 6.99)
- moved C3 0.50 mm to (7.65, 7.17)
- moved C2 0.45 mm to (15.2, 3.20)
- moved U1 0.45 mm to (13.9, 7.00)
- moved TP1 0.40 mm to (12.6, 3.80)
Connections:
- net N$6 renamed EN
- net N$7 renamed BP
Routing:
- net GND: track 20.3 -> 0.00 mm, vias 12 -> 16
- net 3.3V: track 30.2 -> 37.4 mm
- net VBUS: track 11.3 -> 10.6 mm
