File: atmega328p-example/minimal-atmega328p-arduino.brd (EAGLE design)
At the start: 100 x 40 mm, 39 parts, among them J1 3x2 M, J2 1x6 M, J3 629105136821, J4 POWER_JACK, Q1 PMV45EN2R, SW1 !RESET, U1 NCP1117ST50T3G, U4 ATMEGA328P-PU, X1 16 MHz

Commit message: Eeek! Bad cap values for the crystal oscillator. Changed from 18pF to 30 pF based on 18 pF load cap and 0805 capacitors.
Parts:
- C7, C8: value 18p -> 30p
Changed lines of the file:
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@@
 </element>
 <element name="X1" library="SparkFun-Clocks" library_urn="urn:adsk.eagle:library:511" package="HC49UP" package3d_urn="urn:adsk.eagle:package:37513/1" value="16 MHz" x="51" y="26.1" smashed="yes" rot="R180">
+<attribute name="DESC" value="CRYSTAL 16.000 MHZ 18PF SMD" x="51" y="26.1" size="1.778" layer="27" rot="R180" display="off"/>
 <attribute name="MFR" value="ECS" x="51" y="26.1" size="1.778" layer="27" rot="R180" display="off"/>
 <attribute name="MPN" value="ECS-160-18-5PX-TR" x="51" y="26.1" size="1.778" layer="27" rot="R180" display="off"/>
@@
 <attribute name="VALUE" x="51" y="28.767" size="0.6096" layer="27" font="vector" ratio="20" rot="R180" align="top-center"/>
 </element>
-<element name="C7" library="rcl" library_urn="urn:adsk.eagle:library:334" package="C0805K" package3d_urn="urn:adsk.eagle:package:23681/2" value="18p" x="54.8" y="30" smashed="yes" rot="R180">
+<element name="C7" library="rcl" library_urn="urn:adsk.eagle:library:334" package="C0805K" package3d_urn="urn:adsk.eagle:package:23681/2" value="30p" x="54.8" y="30" smashed="yes" rot="R180">
+<attribute name="DESC" value="CAP CER 30PF 50V C0G/NP0 0805" x="54.8" y="30" size="1.778" layer="27" rot="R180" display="off"/>
 <attribute name="MFR" value="Samsung" x="54.8" y="30" size="1.778" layer="27" rot="R180" display="off"/>
 <attribute name="MPN" value="CL21C180JBANNNC" x="54.8" y="30" size="1.778" layer="27" rot="R180" display="off"/>
@@
 <attribute name="VALUE" x="56.07" y="32.54" size="1.27" layer="27" rot="R180"/>
 </element>
-<element name="C8" library="rcl" library_urn="urn:adsk.eagle:library:334" package="C0805K" package3d_urn="urn:adsk.eagle:package:23681/2" value="18p" x="47.2" y="30.01" smashed="yes">
+<element name="C8" library="rcl" library_urn="urn:adsk.eagle:library:334" package="C0805K" package3d_urn="urn:adsk.eagle:package:23681/2" value="30p" x="47.2" y="30.01" smashed="yes">
+<attribute name="DESC" value="CAP CER 30PF 50V C0G/NP0 0805" x="47.2" y="30.01" size="1.778" layer="27" display="off"/>
 <attribute name="MFR" value="Samsung" x="47.2" y="30.01" size="1.778" layer="27" display="off"/>
-<attribute name="MPN" value="CL21C180JBANNNC" x="47.2" y="30.01" size="1.778" layer="27" display="off"/>
+<attribute name="MPN" value="CL21C300JBANNNC" x="47.2" y="30.01" size="1.778" layer="27" display="off"/>
 <attribute name="NAME" x="46.73" y="31.18" size="0.625" layer="25" font="vector" ratio="20"/>
 <attribute name="POPULARITY" value="52" x="47.2" y="30.01" size="1.778" layer="27" display="off"/>
